File: C024926-Adapter.kicad_pcb (KiCad board)
At the start: 2 copper layers, 18 x 36.4 mm, 7 parts, among them J1 Conn_01x14, J2 Conn_01x14, U1 28C256, U2 74AHCT1G04

Commit message: fix link
Other:
- board text added: "https://github.com/ smesgr9000/C024926-Adapter Rev 2"
- board text removed: "https://github.com/ smesgr9000/C024826-Adapter Rev 2"
Changed lines of the file:
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@@
     (effects (font (size 0.5 0.5) (thickness 0.1) bold) (justify left bottom mirror))
   )
-  (gr_text "https://github.com/\nsmesgr9000/C024826-Adapter\nRev 2" (at 160.02 81.7) (layer "B.SilkS")
+  (gr_text "https://github.com/\nsmesgr9000/C024926-Adapter\nRev 2" (at 160.02 81.7) (layer "B.SilkS")
     (effects (font (size 0.5 0.5) (thickness 0.1)) (justify mirror))
   )

Commit message: update to Kicad 8
Parts:
- J1, J2: moved to B.Cu
- turned J1 to 180 degrees
- turned J2 to 180 degrees
